File: 2023l1-int.kicad_pcb (KiCad board)
At the start: 2 copper layers, 185 x 188.1 mm, 134 parts, among them IC1 STM32F103CBTx, IC2 SN74LVC2G04DBVTG4, IC3 SN74LVC2G04DBVTG4, J1 52610-1433, J2 XT30, J3 PGMR, J4 FL, J5 FR, J6 BL, J7 BR, J8 XT60, Q1 STP75NF75, Q2 AO3400A, SW1 STM RST, SW2 L SW, SW3 M SW, U2 CD74HC4067SM, U4 CD74HC4067SM, U5 VNH5050A-E, U6 VNH5050A-E, U7 VNH5050A-E, U8 VNH5050A-E, Y1 8Mhz

Commit message: mux wiring done
Parts:
- moved R31 13.7 mm to (113.7, 90.6), turned to 180 degrees
- moved Q2 7.74 mm to (113.7, 87.6), turned to 90 degrees
- moved C7 6.40 mm to (113.3, 79.6)
- moved R35 6.40 mm to (117.1, 79.6)
- moved R36 6.40 mm to (109.5, 79.6)
- moved R39 5.80 mm to (109.5, 86.6)
- moved Q1 2.75 mm to (113.7, 83.6)
Connections:
- IC1 pad 12: /SOL -> unconnected-(IC1-PA2-Pad12)
- IC1 pad 29: unconnected-(IC1-PA8-Pad29) -> /Sol
Routing:
- net Net-(Q2-D): track 8.53 -> 0.00 mm
- net +12V: track 5.20 -> 0.00 mm
- net Net-(Q1-Pad1): track 2.53 -> 0.00 mm
- net Net-(C7-Pad1): track 2.20 -> 0.00 mm
- net /Sol: track 2.07 -> 0.00 mm
