File: 2023l1-int.kicad_pcb (KiCad board)
At the start: 2 copper layers, 185 x 188.1 mm, 133 parts, among them IC1 STM32F103CBTx, IC2 SN74LVC2G04DBVTG4, IC3 SN74LVC2G04DBVTG4, J1 52610-1433, J2 XT30, J3 PGMR, J4 FL, J5 FR, J6 BL, J7 BR, J8 XT60, Q1 STP75NF75, Q2 AO3400A, SW1 STM RST, SW3 M SW, U2 CD74HC4067SM, U4 CD74HC4067SM, U5 VNH5050A-E, U6 VNH5050A-E, U7 VNH5050A-E, U8 VNH5050A-E, Y1 8Mhz

Commit message: done
Parts:
- moved C11 0.99 mm to (102.7, 97.1)
Routing:
- net +48V: track 30.5 -> 31.5 mm
Changed lines of the file:
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@@
     (fp_arc (start -4.3 2.387868) (mid -4.512132 2.3) (end -4.6 2.087868)
       (stroke (width 0.1) (type default)) (layer "F.SilkS"))
-    (fp_arc (start 4.3 -2.393934) (mid 4.512144 -2.306068) (end 4.6 -2.093934)
+    (fp_arc (start 4.3 -2.393934) (mid 4.512109 -2.306062) (end 4.6 -2.093934)
       (stroke (width 0.1) (type default)) (layer "F.SilkS"))
-    (fp_arc (start 4.6 2.093934) (mid 4.512131 2.306063) (end 4.3 2.393934)
+    (fp_arc (start 4.6 2.093934) (mid 4.512131 2.306067) (end 4.3 2.393934)
       (stroke (width 0.1) (type default)) (layer "F.SilkS"))
     (fp_line (start -4.6 -2.4) (end 4.6 -2.4)
@@
     (fp_arc (start -4.3 2.387868) (mid -4.512132 2.3) (end -4.6 2.087868)
       (stroke (width 0.1) (type default)) (layer "F.SilkS"))
-    (fp_arc (start 4.3 -2.393934) (mid 4.512144 -2.306068) (end 4.6 -2.093934)
+    (fp_arc (start 4.3 -2.393934) (mid 4.512109 -2.306062) (end 4.6 -2.093934)
       (stroke (width 0.1) (type default)) (layer "F.SilkS"))
-    (fp_arc (start 4.6 2.093934) (mid 4.512131 2.306063) (end 4.3 2.393934)
+    (fp_arc (start 4.6 2.093934) (mid 4.512131 2.306067) (end 4.3 2.393934)
       (stroke (width 0.1) (type default)) (layer "F.SilkS"))
     (fp_line (start -4.6 -2.4) (end 4.6 -2.4)
@@
     (fp_arc (start -4.3 2.387868) (mid -4.512132 2.3) (end -4.6 2.087868)
       (stroke (width 0.1) (type default)) (layer "F.SilkS"))
-    (fp_arc (start 4.3 -2.393934) (mid 4.512144 -2.306068) (end 4.6 -2.093934)
+    (fp_arc (start 4.3 -2.393934) (mid 4.512109 -2.306062) (end 4.6 -2.093934)
       (stroke (width 0.1) (type default)) (layer "F.SilkS"))
-    (fp_arc (start 4.6 2.093934) (mid 4.512131 2.306063) (end 4.3 2.393934)
+    (fp_arc (start 4.6 2.093934) (mid 4.512131 2.306067) (end 4.3 2.393934)
       (stroke (width 0.1) (type default)) (layer "F.SilkS"))
     (fp_line (start -4.6 -2.4) (end 4.6 -2.4)
@@
   )
   (footprint "footprints:CAPAE1030X1270N" (layer "F.Cu")
-    (at 103.68041 96.993602 -90)
+    (at 102.7 97.1 -90)
     (descr "10mmx12.7mm")
     (tags "Capacitor Polarised")
@@
     (fp_arc (start -4.3 2.387868) (mid -4.512132 2.3) (end -4.6 2.087868)
       (stroke (width 0.1) (type default)) (layer "F.SilkS"))
-    (fp_arc (start 4.3 -2.393934) (mid 4.512144 -2.306068) (end 4.6 -2.093934)
+    (fp_arc (start 4.3 -2.393934) (mid 4.512109 -2.306062) (end 4.6 -2.093934)
       (stroke (width 0.1) (type default)) (layer "F.SilkS"))
-    (fp_arc (start 4.6 2.093934) (mid 4.512131 2.306063) (end 4.3 2.393934)
+    (fp_arc (start 4.6 2.093934) (mid 4.512131 2.306067) (end 4.3 2.393934)
       (stroke (width 0.1) (type default)) (layer "F.SilkS"))
     (fp_line (start -4.6 -2.4) (end 4.6 -2.4)
@@
   (segment (start 102.8804 21.7936) (end 102.8904 21.8036) (width 0.3) (layer "F.Cu") (net 96))
   (segment (start 102.8904 21.8036) (end 105.8804 21.8036) (width 0.3) (layer "F.Cu") (net 96))
-  (segment (start 111.1804 92.793602) (end 103.73041 92.793602) (width 3) (layer "F.Cu") (net 97))
-  (segment (start 103.73041 92.793602) (end 103.68041 92.743602) (width 3) (layer "F.Cu") (net 97))
   (segment (start 97.2804 78.27359) (end 106.06041 87.0536) (width 3) (layer "F.Cu") (net 97))
+  (segment (start 102.756398 92.793602) (end 102.7 92.85) (width 3) (layer "F.Cu") (net 97))
   (segment (start 97.2804 75.593602) (end 97.2804 78.27359) (width 3) (layer "F.Cu") (net 97))
+  (segment (start 111.1804 92.793602) (end 102.756398 92.793602) (width 3) (layer "F.Cu") (net 97))
   (segment (start 106.06041 87.673612) (end 111.1804 92.793602) (width 3) (layer "B.Cu") (net 97))
   (segment (start 106.06041 87.0536) (end 106.06041 87.673612) (width 3) (layer "B.Cu") (net 97))
