File: 2023l1-int.kicad_sch (KiCad schematic)
At the start: 133 parts, among them J1 52610-1433, J8 XT60, Q1 STP75NF75

Commit message: left with msw
Connections:
- net !BL DIR: now also U?.15 (INA); no longer U?.22 (INB)
- net !BR DIR: now also U?.22 (INB); no longer U?.15 (INA)
- net !FL DIR: now also U?.22 (INB); no longer U?.15 (INA)
- net !FR DIR: now also U?.15 (INA); no longer U?.22 (INB)
- net BL DIR: now also U?.22 (INB); no longer U?.15 (INA)
- net BR DIR: now also U?.15 (INA); no longer U?.22 (INB)
- net FL DIR: now also U?.15 (INA); no longer U?.22 (INB)
- net FR DIR: now also U?.22 (INB); no longer U?.15 (INA)
- net RX: now also U?.13 (PA3); no longer U?.30 (PA9)
- net TX: now also U?.12 (PA2); no longer U?.31 (PA10)
- no-connect marks 30 -> 28
